File: board/Pulsar Buddy.brd (EAGLE design)
At the start: 144.8 x 53.3 mm, 54 parts, among them IC1 7805TV, T1 2N2222, T2 2N2222, T3 2N2222, T4 2N2222, T5 2N2222, T6 2N2222

Commit message: rev B board
Parts:
- removed BR1: W005G-E4_51, SamacSys:W005G-E4/51
- removed C1: 22u, rcl:E3,5-8
- removed C2, C3: 100n, rcl:C025-024X044
- removed IC1: 7805TV, linear:TO220V
- added C1A: 330n, rcl:C025-024X044
- added C1B: 10u, rcl:E5-5
- added C2A: 100n, rcl:C025-024X044
- added C2B: 22u, rcl:E5-5
- added D4, D5, D6: (no value), diode:DO35-7
- added D7, D8, D9: 1N4004, diode:DO41-10
- added IC2: UA78M33CKCSTO-220, pb extras:TO220H
- added R17, R18: 100kΩ, rcl:0204/7
- added R19, R20: 33kΩ, rcl:0204/7
- D1, D2: value 1N4004 -> (none); device diode:DO41-10 -> diode:DO35-7
- D3: value 1N4148DO35-7 -> (none)
- R1, R15, R4: value 100kΩ -> 1kΩ
- R10, R13: value 100kΩ -> 10kΩ
- R11: value 1kΩ -> 10kΩ
- R12, R9: value 3.3kΩ -> 10kΩ
- R14: value 33kΩ -> 10kΩ
- R16: value 33kΩ -> 1kΩ
- R2: value 10kΩ -> 1kΩ
- R3: value 3.3kΩ -> 1kΩ
- R5: value 10kΩ -> 2.2kΩ
- R6: value 3.3kΩ -> 2.2kΩ
- R7: value 100kΩ -> 2.2kΩ
- R8: value 1kΩ -> 2.2kΩ
- moved R4 83.2 mm to (20.3, 21.6), turned to 90 degrees
- moved R11 82.3 mm to (118.1, 33.0), flipped to the bottom
- moved R14 72.6 mm to (41.9, 45.7), turned to 270 degrees
- moved R16 72.2 mm to (36.8, 45.7), turned to 270 degrees
- moved R8 58.8 mm to (88.9, 14.0), turned to 180 degrees
- moved R3 55.3 mm to (33.0, 21.6), turned to 90 degrees
- moved R1 53.1 mm to (58.4, 21.6), turned to 90 degrees
- moved R5 52.3 mm to (88.3, 21.6), turned to 180 degrees
- moved D3 36.9 mm to (76.2, 12.7)
- moved R13 35.9 mm to (44.5, 45.7)
- moved D1 32.4 mm to (76.2, 25.4)
- moved R9 31.9 mm to (115.6, 31.8), flipped to the bottom, turned to 270 degrees
- moved R7 31.4 mm to (86.4, 16.5), turned to 180 degrees
- moved R12 30.0 mm to (113.0, 34.3), flipped to the bottom, turned to 270 degrees
- moved R15 29.8 mm to (39.4, 45.7)
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- renumbered BAN_CIN to PAD110, BAN_OIN to PAD112, JP2 to JP16, JP3 to JP12, LED_B to LED3, LED_M to LED2, LED_S to LED1, LED_T to LED4, MS2 to MS101, PAD_G1 to PAD_GND, PIN_CIN to PAD109, PIN_OIN to PAD111, VR1 to SW1
Connections:
- removed net +12V_RAW: BR1.4, F1.2
- removed net +5V: C2.1, IC1.3, JP12.3, MS101.26, R12.1, R3.1, R6.1, R9.1
- removed net LED_3V3: JP1.2, R11.1, R2.1, R5.1, R8.1
- new net +10V: D9.C, R5.1, R6.1, R7.1, R8.1
- new net +3V3_LED: JP1.2, R13.1, R14.1, R15.1, R16.1
- new net +5V_CPU: JP12.3, MS101.26
- new net N$37: BAN_S.C, PIN_S.1, R1.2
- new net N$38: BAN_M.C, PIN_M.1, R2.2
- new net N$39: BAN_T.C, PIN_T.1, R4.2
- new net N$40: BAN_B.C, PIN_B.1, R3.2
- net +12V: now also C1A.1, C1B.+, D8.A, IC2.1; no longer C1.+, C3.1, D3.C, IC1.1
- net +3V3: now also C2A.1, C2B.+, IC2.3
- net GND: now also C1A.2, C1B.-, C2A.2, C2B.-, D4.A, D5.A, D6.A, IC2.2, J1.1, JP12.2, MS101.27, R19.2, R20.2; no longer BR1.2, C1.-, C2.2, C3.2, IC1.2, R14.2, R16.2
- net N$10: now also R10.2; no longer R4.2
- net N$11: now also D2.C, R2.1; no longer BAN_M.C, PIN_M.1
- net N$12: now also R15.2; no longer R8.2
- net N$13: now also R11.2; no longer R7.2
- net N$14: now also D3.C, R3.1, R7.2; no longer BAN_B.C, PIN_B.1, R9.2
- net N$15: now also R16.2; no longer R11.2
- net N$16: now also R12.2; no longer R10.2
- net N$17: now also D4.C, R4.1, R8.2; no longer BAN_T.C, PIN_T.1, R12.2
- net N$18: now also D5.C, R17.2, R19.1; no longer D1.C, R13.2, R14.1
- net N$19: now also R18.1; no longer R15.1
- net N$20: now also R17.1; no longer R13.1
- net N$21: now also D6.C, R18.2, R20.1; no longer D2.C, R15.2, R16.1
- net N$36: now also D8.C, D9.A; no longer JP12.2, MS101.27
- net N$4: now also D7.C, F1.2; no longer BR1.3, J1.3
- net N$5: now also D7.A, J1.3; no longer BR1.1, J1.1
- net N$6: now also R13.2; no longer R2.2
- net N$7: now also R14.2; no longer R5.2
- net N$8: now also R9.2; no longer R1.2
- net N$9: now also D1.C, R1.1, R5.2; no longer BAN_S.C, PIN_S.1, R3.2
- net T_BEAT: now also R11.1; no longer R7.1
- net T_MEASURE: now also R10.1; no longer R4.1
- net T_SEQUENCE: now also R9.1; no longer R1.1
- net T_TUPLET: now also R12.1; no longer R10.1
Routing:
- net +5V: track 68.8 -> 0.00 mm
- net N$39: track 0.00 -> 30.9 mm
- net N$37: track 0.00 -> 30.1 mm
- net N$40: track 0.00 -> 29.4 mm
- net N$38: track 0.00 -> 28.2 mm
- net N$17: track 102.2 -> 79.3 mm
- net N$14: track 79.5 -> 58.1 mm
- net N$11: track 69.5 -> 48.2 mm
- net N$9: track 60.0 -> 41.9 mm
- net +10V: track 0.00 -> 17.2 mm
- net +12V_RAW: track 15.1 -> 0.00 mm
- net LED_3V3: track 12.5 -> 0.00 mm
- net +3V3_LED: track 0.00 -> 12.3 mm
- net +3V3: track 93.9 -> 104.5 mm
- net N$4: track 24.1 -> 14.6 mm
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Other:
- board text added: "C"
- board text added: "Clock"
- board text added: "O"
- board text added: "Other"
- board text removed: "> Other"
- board text removed: ">Clock"
