File: board/Pulsar Buddy.brd (EAGLE design)
At the start: 144.8 x 53.3 mm, 64 parts, among them IC2 UA78M33CKCSTO-220, SW1 PEC11R-4220F-S0024, T1 2N2222, T2 2N2222, T3 2N2222, T4 2N2222, T5 2N2222, T6 2N2222

Commit message: rev C. board layout
Parts:
- moved C1B 24.5 mm to (74.9, 45.7), flipped to the bottom
- moved C1A 9.61 mm to (83.2, 49.5)
- moved IC2 6.63 mm to (80.6, 38.1), turned to 225 degrees
- moved C2B 4.84 mm to (89.5, 33.7), flipped to the bottom, turned to 270 degrees
- moved C2A 3.86 mm to (92.1, 40.6), turned to 270 degrees
- moved T3 3.81 mm to (81.3, 26.7), turned to 0 degrees
- moved T4 2.84 mm to (88.9, 26.7), turned to 0 degrees
- moved D1 2.54 mm to (73.7, 25.4)
- moved D2 2.54 mm to (76.2, 22.9)
- moved T1 1.80 mm to (91.4, 8.89), turned to 180 degrees
- moved T6 1.80 mm to (129.5, 7.62), turned to 0 degrees
- moved D3 1.31 mm to (74.9, 12.4)
- moved T2 1.27 mm to (83.8, 8.89), turned to 180 degrees
- moved T5 1.27 mm to (135.9, 3.81), turned to 0 degrees
- moved D4 1.27 mm to (77.5, 10.2)
Routing:
- net +12V: track 57.7 -> 84.4 mm
- net N$13: track 35.0 -> 40.9 mm
- net T_CLK_IN: track 45.2 -> 48.7 mm
- net T_OTHER_IN: track 40.0 -> 43.4 mm
- net +3V3: track 104.5 -> 107.3 mm
- net N$16: track 24.4 -> 27.0 mm
- net N$8: track 37.9 -> 35.8 mm
- net T_MEASURE: track 74.4 -> 76.2 mm
- net T_TUPLET: track 103.5 -> 105.3 mm
- net T_SEQUENCE: track 69.2 -> 71.0 mm
- net T_BEAT: track 96.5 -> 98.3 mm
- net N$18: track 135.0 -> 136.3 mm
- net N$14: track 58.1 -> 59.4 mm
- net N$9: track 41.9 -> 40.9 mm
- net N$17: track 79.3 -> 80.3 mm
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Other:
- board text added: "G"
- board text added: "R"
- board text added: "rev. C"
- board text removed: "rev. B"
