File: board/Pulsar Buddy.sch (EAGLE design)
At the start: 54 parts, among them IC1 7805TV, T1 2N2222, T2 2N2222, T3 2N2222, T4 2N2222, T5 2N2222, T6 2N2222

Commit message: rev B board
Parts:
- removed BR1: W005G-E4_51, SamacSys:W005G-E4_51
- removed C1: 22u, rcl:CPOL-USE3.5-8
- removed C3: 100n, rcl:C-EU025-024X044
- removed IC1: 7805TV, linear:7805TV
- removed LED_B, LED_T: GREEN, led:LED5MM
- removed LED_M, LED_S: RED, led:LED5MM
- added C1A: 330n, rcl:C-EU025-024X044
- added C1B: 10u, rcl:CPOL-USE5-5
- added C2B: 22u, rcl:CPOL-USE5-5
- added D4, D5, D6: (no value), diode:SCHOTTKY-DIODEDO35-7
- added D7, D8, D9: 1N4004, diode:1N4004
- added IC2: UA78M33CKCSTO-220, pb extras:UA78M33CKCSTO-220
- added LED1, LED2: RED, led:LED5MM
- added LED3, LED4: GREEN, led:LED5MM
- added R17, R18: 100kΩ, rcl:R-US_0204/7
- added R19, R20: 33kΩ, rcl:R-US_0204/7
- D1, D2: value 1N4004 -> (none); device diode:1N4004 -> diode:SCHOTTKY-DIODEDO35-7
- D3: value 1N4148DO35-7 -> (none); device diode:1N4148DO35-7 -> diode:SCHOTTKY-DIODEDO35-7
- R1, R15, R4: value 100kΩ -> 1kΩ
- R10, R13: value 100kΩ -> 10kΩ
- R11: value 1kΩ -> 10kΩ
- R12, R9: value 3.3kΩ -> 10kΩ
- R14: value 33kΩ -> 10kΩ
- R16: value 33kΩ -> 1kΩ
- R2: value 10kΩ -> 1kΩ
- R3: value 3.3kΩ -> 1kΩ
- R5: value 10kΩ -> 2.2kΩ
- R6: value 3.3kΩ -> 2.2kΩ
- R7: value 100kΩ -> 2.2kΩ
- R8: value 1kΩ -> 2.2kΩ
- renumbered BAN_CIN to PAD110, BAN_OIN to PAD112, C2 to C2A, JP2 to JP16, JP3 to JP12, MS2 to MS101, PAD_G1 to PAD_GND, PIN_CIN to PAD109, PIN_OIN to PAD111, VR1 to SW1
Connections:
- removed net +12V_RAW: BR1.+, F1.2
- removed net +5V: C2A.1, IC1.VO, JP12.3, MS101.USB, R12.1, R3.1, R6.1, R9.1
- removed net LED_3V3: JP1.2, R11.1, R2.1, R5.1, R8.1
- new net +10V: D9.C, R5.1, R6.1, R7.1, R8.1
- new net +3V3_LED: JP1.2, R13.1, R14.1, R15.1, R16.1
- new net +5V_CPU: JP12.3, MS101.USB
- new net N$37: BAN_S.P, PIN_S.P, R1.2
- new net N$38: BAN_M.P, PIN_M.P, R2.2
- new net N$39: BAN_T.P, PIN_T.P, R4.2
- new net N$40: BAN_B.P, PIN_B.P, R3.2
- net +12V: now also C1A.1, C1B.+, D8.A, IC2.IN; no longer C1.+, C3.1, D3.C, IC1.VI
- net +3V3: now also C2A.1, C2B.+, IC2.OUT
- net GND: now also C1A.2, C1B.-, C2B.-, D4.A, D5.A, D6.A, IC2.GND, J1.1, JP12.2, MS101.EN, R19.2, R20.2; no longer BR1.-, C1.-, C3.2, IC1.GND, R14.2, R16.2
- net N$10: now also R10.2; no longer R4.2
- net N$11: now also D2.C, R2.1; no longer BAN_M.P, PIN_M.P
- net N$12: now also LED3.A, R15.2; no longer LED_B.A, R8.2
- net N$13: now also R11.2; no longer R7.2
- net N$14: now also D3.C, R3.1, R7.2; no longer BAN_B.P, PIN_B.P, R9.2
- net N$15: now also LED4.A, R16.2; no longer LED_T.A, R11.2
- net N$16: now also R12.2; no longer R10.2
- net N$17: now also D4.C, R4.1, R8.2; no longer BAN_T.P, PIN_T.P, R12.2
- net N$18: now also D5.C, R17.2, R19.1; no longer D1.C, R13.2, R14.1
- net N$19: now also R18.1; no longer R15.1
- net N$20: now also R17.1; no longer R13.1
- net N$21: now also D6.C, R18.2, R20.1; no longer D2.C, R15.2, R16.1
- net N$36: now also D8.C, D9.A; no longer JP12.2, MS101.EN
- net N$4: now also D7.C, F1.2; no longer BR1.~_2, J1.3
- net N$5: now also D7.A, J1.3; no longer BR1.~_1, J1.1
- net N$6: now also LED1.A, R13.2; no longer LED_S.A, R2.2
- net N$7: now also LED2.A, R14.2; no longer LED_M.A, R5.2
- net N$8: now also R9.2; no longer R1.2
- net N$9: now also D1.C, R1.1, R5.2; no longer BAN_S.P, PIN_S.P, R3.2
- net T_BEAT: now also LED3.C, R11.1; no longer LED_B.C, R7.1
- net T_MEASURE: now also LED2.C, R10.1; no longer LED_M.C, R4.1
- net T_SEQUENCE: now also LED1.C, R9.1; no longer LED_S.C, R1.1
- net T_TUPLET: now also LED4.C, R12.1; no longer LED_T.C, R10.1
Other:
- note added: "Either: A - UA78M33 linear regulator B - VXO7803-500 switching regulator"
- note added: "Install only --A or --B capacitors, matching the regulator choice."
- note added: "PTC resettable fuse such as: Bournes MF-R020 Bel Fuse 0ZRR0020FF1E"
- moved on the sheet: BAN_B, BAN_M, BAN_S, BAN_T, F1, PIN_B, PIN_M, PIN_S, PIN_T, R1, R10, R11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
